Commit message: Fix slave's URDF reference

File: mimic_support/urdf/mimic_slave_v2.xacro (robot description, xacro)
@@ -22,23 +22,4 @@
                 <geometry>
                 <mesh filename="package://mimic_support/meshes/collision/ktig_eef_v2.stl" scale="0.001 0.001 0.001"/>
-                </geometry>
-            </collision>
-        </link>
-        <link name="base_10">
-            <inertial>
-                <origin xyz="0 0 0" rpy="0 0 0"/>
-                <mass value="2"/>
-                <inertia ixx="0.01" ixy="0" ixz="0" iyy="0.01" iyz="0" izz="0.01" />
-            </inertial>
-            <visual>
-                <origin xyz="0 0 0" rpy="0 0 0"/>
-                <geometry>
-                <mesh filename="package://mimic_support/meshes/visual/positioner.dae" scale="0.001 0.001 0.001"/>
-                </geometry>
-            </visual>
-            <collision>
-                <origin xyz="0 0 0" rpy="0 0 0"/>
-                <geometry>
-                <mesh filename="package://mimic_support/meshes/collision/positioner.stl" scale="0.001 0.001 0.001"/>
                 </geometry>
             </collision>
@@ -70,8 +51,3 @@
             <!-- <origin xyz="0.121 0.05578 0.5307" rpy="${radians(0)} ${radians(-19.95)} ${radians(24.259)}" /> -->
         </joint>
-        <joint name="world-base_10" type="fixed">
-            <parent link="world" />
-            <child link="base_10" />
-            <origin xyz="4.6629 2.5080 -8.7763" rpy="${radians(0.58)} ${radians(0.15)} ${radians(0.35)}" />
-        </joint>
     </robot>
