Commit message: Change configuration files

File: mimic_support/urdf/mimic_master.xacro (robot description, xacro)
@@ -1,5 +1,5 @@
 <?xml version="1.0"?>
     <robot name="mimic_slave" xmlns:xacro="http://ros.org/wiki/xacro">
-        <xacro:property name="prefix" value="master_" />
+        <xacro:property name="prefix" value="" />
         <xacro:include filename="positioner_macro.xacro"/>
         <xacro:positioner prefix="${prefix}"/>

File: mimic_support/urdf/mimic_slave.xacro (robot description, xacro)
@@ -1,5 +1,5 @@
 <?xml version="1.0"?>
     <robot name="mimic_slave" xmlns:xacro="http://ros.org/wiki/xacro">
-        <xacro:property name="prefix" value="slave_" />
+        <xacro:property name="prefix" value="" />
         <xacro:include filename="gantry_macro.xacro"/>
         <xacro:gantry  prefix="${prefix}"/>
