Commit message: Fix slave and master URDF

File: mimic_support/urdf/gantry_macro.xacro (robot description, xacro)
@@ -81,5 +81,5 @@
                 <child link="${prefix}gantry_x"/>
                 <axis xyz="1 0 0"/>
-                <limit effort="0" lower="-0.011" upper="3" velocity="${radians(156)}"/>
+                <limit effort="21.9" lower="-0.011" upper="3.0" velocity="0.83"/>
             </joint>
             <joint name="${prefix}joint_e2" type="prismatic">
@@ -88,5 +88,5 @@
                 <child link="${prefix}gantry_y"/>
                 <axis xyz="0 1 0"/>
-                <limit effort="0" lower="-0.015" upper="2.25" velocity="${radians(156)}"/>
+                <limit effort="24.4" lower="-0.015" upper="2.25" velocity="1.25"/>
             </joint>
             <joint name="${prefix}joint_e3" type="prismatic">
@@ -95,5 +95,5 @@
                 <child link="${prefix}gantry_z"/>
                 <axis xyz="0 0 -1"/>
-                <limit effort="0" lower="-0.011" upper="2.6" velocity="${radians(156)}"/>
+                <limit effort="52.6" lower="-0.011" upper="2.6" velocity="0.75"/>
             </joint>
         </xacro:macro>

File: mimic_support/urdf/mimic_master.xacro (robot description, xacro)
@@ -12,5 +12,8 @@
             <parent link="world" />
             <child link="positioner_frame" />
-            <origin xyz="0.87144 1.19321 0.3000" rpy="0.0 0.0 ${radians(50)}" />
+            <!-- <origin xyz="0.8714369 1.1932095 0.3000" rpy="0.0 0.0 ${radians(50)}" /> -->
+            <!-- <origin xyz="1.1932095 0.8714369 0.3000" rpy="0.0 0.0 ${radians(50)}" /> -->
+            <!-- <origin xyz="1.1932095 1.171426018 0.3000" rpy="0.0 0.0 ${radians(50)}" /> -->
+            <origin xyz="0.0994209235 1.4742 0.3000" rpy="0.0 0.0 ${radians(50)}" />
         </joint>
     </robot>

File: mimic_support/urdf/mimic_slave_v2.xacro (robot description, xacro)
@@ -35,6 +35,6 @@
             <origin xyz="0.0 0.0 0.0" rpy="${radians(0.641)} 0.0 0.0" />
         </joint>
-        <joint name="robroot-gantry_joint" type="fixed">
-            <parent link="robroot" />
+        <joint name="ersysroot-gantry_joint" type="fixed">
+            <parent link="ersysroot" />
             <child link="gantry_frame" />
             <origin xyz="0.0 0.0 0.0" rpy="0.0 0.0 0.0" />

File: mimic_support/urdf/positioner_macro.xacro (robot description, xacro)
@@ -62,5 +62,5 @@
                 <child link="${prefix}e1"/>
                 <axis xyz="1 0 0"/>
-                <limit effort="0" lower="-0.011" upper="3" velocity="${radians(156)}"/>
+                <limit effort="21.9" lower="-2.5" upper="117.5" velocity="0.714"/>
             </joint>
             <joint name="${prefix}joint_e2" type="revolute">
@@ -69,5 +69,5 @@
                 <child link="${prefix}e2"/>
                 <axis xyz="0 0 1"/>
-                <limit effort="0" lower="-0.015" upper="2.25" velocity="${radians(156)}"/>
+                <limit effort="21.9" lower="-1800" upper="1800" velocity="0.2575"/>
             </joint>
         </xacro:macro>

Commit message: Enables whole cell control

File: mimic_support/urdf/gantry_macro.xacro (robot description, xacro)
@@ -7,5 +7,5 @@
                     <origin xyz="0 0 0" rpy="0 0 0"/>
                     <geometry>
-                    <mesh filename="package://mimic_support/meshes/visual/gantry_frame_c.dae" scale="0.001 0.001 0.001"/>
+                    <mesh filename="package://mimic_support/meshes/visual/gantry_fixed.dae" scale="0.001 0.001 0.001"/>
                     </geometry>
                 </visual>
@@ -13,5 +13,5 @@
                     <origin xyz="0 0 0" rpy="0 0 0"/>
                     <geometry>
-                    <mesh filename="package://mimic_support/meshes/collision/gantry_frame_c.stl" scale="0.001 0.001 0.001"/>
+                    <mesh filename="package://mimic_support/meshes/collision/gantry_fixed.stl" scale="0.001 0.001 0.001"/>
                     </geometry>
                 </collision>
@@ -26,5 +26,5 @@
                     <origin xyz="0 0 0" rpy="0 0 0"/>
                     <geometry>
-                    <mesh filename="package://mimic_support/meshes/visual/gantry_x_c.dae" scale="0.001 0.001 0.001"/>
+                    <mesh filename="package://mimic_support/meshes/visual/gantry_x.dae" scale="0.001 0.001 0.001"/>
                     </geometry>
                 </visual>
@@ -32,5 +32,5 @@
                     <origin xyz="0 0 0" rpy="0 0 0"/>
                     <geometry>
-                    <mesh filename="package://mimic_support/meshes/collision/gantry_x_c.stl" scale="0.001 0.001 0.001"/>
+                    <mesh filename="package://mimic_support/meshes/collision/gantry_x.stl" scale="0.001 0.001 0.001"/>
                     </geometry>
                 </collision>
@@ -45,5 +45,5 @@
                     <origin xyz="0 0 0" rpy="0 0 0"/>
                     <geometry>
-                    <mesh filename="package://mimic_support/meshes/visual/gantry_y_c.dae" scale="0.001 0.001 0.001"/>
+                    <mesh filename="package://mimic_support/meshes/visual/gantry_y.dae" scale="0.001 0.001 0.001"/>
                     </geometry>
                 </visual>
@@ -51,5 +51,5 @@
                     <origin xyz="0 0 0" rpy="0 0 0"/>
                     <geometry>
-                    <mesh filename="package://mimic_support/meshes/collision/gantry_y_c.stl" scale="0.001 0.001 0.001"/>
+                    <mesh filename="package://mimic_support/meshes/collision/gantry_y.stl" scale="0.001 0.001 0.001"/>
                     </geometry>
                 </collision>
@@ -64,5 +64,5 @@
                     <origin xyz="0 0 0" rpy="0 0 0"/>
                     <geometry>
-                    <mesh filename="package://mimic_support/meshes/visual/gantry_z_c.dae" scale="0.001 0.001 0.001"/>
+                    <mesh filename="package://mimic_support/meshes/visual/gantry_z.dae" scale="0.001 0.001 0.001"/>
                     </geometry>
                 </visual>
@@ -70,5 +70,5 @@
                     <origin xyz="0 0 0" rpy="0 0 0"/>
                     <geometry>
-                    <mesh filename="package://mimic_support/meshes/collision/gantry_z_c.stl" scale="0.001 0.001 0.001"/>
+                    <mesh filename="package://mimic_support/meshes/collision/gantry_z.stl" scale="0.001 0.001 0.001"/>
                     </geometry>
                 </collision>
@@ -77,5 +77,5 @@
             <!-- joint e1 (E1) -->
             <joint name="${prefix}joint_e1" type="prismatic">
-                <origin xyz="0 0 0" rpy="0 0 0"/>
+                <origin xyz="0.011 0 0" rpy="0 0 0"/>
                 <parent link="${prefix}gantry_frame"/>
                 <child link="${prefix}gantry_x"/>
@@ -84,5 +84,5 @@
             </joint>
             <joint name="${prefix}joint_e2" type="prismatic">
-                <origin xyz="0 0 0" rpy="0 0 0"/>
+                <origin xyz="0 0.015 0" rpy="0 0 0"/>
                 <parent link="${prefix}gantry_x"/>
                 <child link="${prefix}gantry_y"/>
@@ -91,5 +91,5 @@
             </joint>
             <joint name="${prefix}joint_e3" type="prismatic">
-                <origin xyz="0 0 0" rpy="0 0 0"/>
+                <origin xyz="0 0 0.011" rpy="0 0 0"/>
                 <parent link="${prefix}gantry_y"/>
                 <child link="${prefix}gantry_z"/>

File: mimic_support/urdf/mimic_master.xacro (robot description, xacro)
@@ -1,15 +1,18 @@
 <?xml version="1.0"?>
     <robot name="mimic_slave" xmlns:xacro="http://ros.org/wiki/xacro">
-        <xacro:include filename="positioner.xacro"/>
-        <xacro:include filename="$(find kuka_kr20_support)/urdf/kr20_r1810_2.xacro" />
-        <link name="world" />
-        <joint name="world-kr20" type="fixed">
-            <parent link="world" />
-            <child link="base_link" />
+        <xacro:property name="prefix" value="master_" />
+        <xacro:include filename="positioner_macro.xacro"/>
+        <xacro:positioner prefix="${prefix}"/>
+        <xacro:include filename="$(find kuka_kr20_support)/urdf/kr20_r1810_2_macro.xacro" />
+        <xacro:kuka_kr20_r1810_2 prefix="${prefix}"/>
+        <link name="${prefix}world" />
+        <joint name="${prefix}world-${prefix}kr20_joint" type="fixed">
+            <parent link="${prefix}world" />
+            <child link="${prefix}base_link" />
             <origin xyz="0.0 0.0 0.0" rpy="0.0 0.0 0.0" />
         </joint>
-        <joint name="world-positioner" type="fixed">
-            <parent link="world" />
-            <child link="positioner_frame" />
+        <joint name="${prefix}world-${prefix}positioner_joint" type="fixed">
+            <parent link="${prefix}world" />
+            <child link="${prefix}positioner_frame" />
             <!-- <origin xyz="0.8714369 1.1932095 0.3000" rpy="0.0 0.0 ${radians(50)}" /> -->
             <!-- <origin xyz="1.1932095 0.8714369 0.3000" rpy="0.0 0.0 ${radians(50)}" /> -->

File: mimic_support/urdf/mimic_slave.xacro (robot description, xacro)
@@ -1,8 +1,11 @@
 <?xml version="1.0"?>
     <robot name="mimic_slave" xmlns:xacro="http://ros.org/wiki/xacro">
-        <xacro:include filename="gantry.xacro"/>
-        <xacro:include filename="$(find kuka_kr16_support)/urdf/kr16_2.xacro" />
-        <link name="world" />
-        <link name="ktig_eef">
+        <xacro:property name="prefix" value="slave_" />
+        <xacro:include filename="gantry_macro.xacro"/>
+        <xacro:gantry  prefix="${prefix}"/>
+        <xacro:include filename="$(find kuka_kr16_support)/urdf/kr16_2_macro.xacro"/>
+        <xacro:kuka_kr16_2  prefix="${prefix}"/>
+        <link name="${prefix}world" />
+        <link name="${prefix}ktig_eef">
             <inertial>
                 <origin xyz="0 0 0" rpy="0 0 0"/>
@@ -23,17 +26,17 @@
             </collision>
         </link>
-        <joint name="world-gantry_joint" type="fixed">
-            <parent link="world" />
-            <child link="gantry_frame" />
+        <joint name="${prefix}world-${prefix}gantry_joint" type="fixed">
+            <parent link="${prefix}world" />
+            <child link="${prefix}gantry_frame" />
             <origin xyz="0.0 0.0 0.0" rpy="0.0 0.0 0.0" />
         </joint>
-        <joint name="gantry-kr16_joint" type="fixed">
-            <parent link="gantry_z" />
-            <child link="base_link" />
+        <joint name="${prefix}gantry-${prefix}kr16_joint" type="fixed">
+            <parent link="${prefix}gantry_z" />
+            <child link="${prefix}base_link" />
             <origin xyz="0.0 0.0 0.0" rpy="${pi} 0.0 0.0" />
         </joint>
-        <joint name="kr16-ktig_joint" type="fixed">
-            <parent link="tool0" />
-            <child link="ktig_eef" />
+        <joint name="${prefix}kr16-${prefix}ktig_joint" type="fixed">
+            <parent link="${prefix}tool0" />
+            <child link="${prefix}ktig_eef" />
             <origin xyz="0.0811 0.04116 0.4408" rpy="${radians(-179.61)} ${radians(-41.39)} ${radians(-153.95)}" />
             <!-- <origin xyz="0.121 0.05578 0.5307" rpy="${radians(0)} ${radians(-19.95)} ${radians(24.259)}" /> -->

Commit message: Add torque values into gantry URDF

File: mimic_support/urdf/gantry_macro.xacro (robot description, xacro)
@@ -81,5 +81,5 @@
                 <child link="${prefix}gantry_x"/>
                 <axis xyz="1 0 0"/>
-                <limit effort="21.9" lower="-0.011" upper="3.0" velocity="0.83"/>
+                <limit effort="12100" lower="-0.011" upper="3.0" velocity="0.83"/>
             </joint>
             <joint name="${prefix}joint_e2" type="prismatic">
@@ -88,5 +88,5 @@
                 <child link="${prefix}gantry_y"/>
                 <axis xyz="0 1 0"/>
-                <limit effort="24.4" lower="-0.015" upper="2.25" velocity="1.25"/>
+                <limit effort="25000" lower="-0.015" upper="2.25" velocity="1.25"/>
             </joint>
             <joint name="${prefix}joint_e3" type="prismatic">
@@ -95,5 +95,5 @@
                 <child link="${prefix}gantry_z"/>
                 <axis xyz="0 0 -1"/>
-                <limit effort="52.6" lower="-0.011" upper="2.6" velocity="0.75"/>
+                <limit effort="79500" lower="-0.011" upper="2.6" velocity="0.75"/>
             </joint>
         </xacro:macro>

Commit message: Limit external axis velocity limit

File: mimic_support/urdf/gantry_macro.xacro (robot description, xacro)
@@ -81,5 +81,5 @@
                 <child link="${prefix}gantry_x"/>
                 <axis xyz="1 0 0"/>
-                <limit effort="12100" lower="-0.011" upper="3.0" velocity="0.83"/>
+                <limit effort="12" lower="-0.011" upper="3.0" velocity="0.1"/>
             </joint>
             <joint name="${prefix}joint_e2" type="prismatic">
@@ -88,5 +88,5 @@
                 <child link="${prefix}gantry_y"/>
                 <axis xyz="0 1 0"/>
-                <limit effort="25000" lower="-0.015" upper="2.25" velocity="1.25"/>
+                <limit effort="25" lower="-0.015" upper="2.25" velocity="0.4"/>
             </joint>
             <joint name="${prefix}joint_e3" type="prismatic">
@@ -95,5 +95,5 @@
                 <child link="${prefix}gantry_z"/>
                 <axis xyz="0 0 -1"/>
-                <limit effort="79500" lower="-0.011" upper="2.6" velocity="0.75"/>
+                <limit effort="79" lower="-0.011" upper="2.6" velocity="0.1"/>
             </joint>
         </xacro:macro>
