Commit message: new positions

File: mimic_support/urdf/mimic_v2.xacro (robot description, xacro)
@@ -36,5 +36,6 @@
             <parent link="world" />
             <child link="${prefix_slave}gantry_frame" />
-            <origin xyz="0.0 0.0 0.0" rpy="0.0 0.0 0.0" />
+            <!-- <origin xyz="3.04787 1.209 -4.974558" rpy="0.0 ${radians(0.038)} ${radians(0.211)}" /> -->
+            <origin xyz="3.05881 1.224 -4.98539" rpy="0.0 ${radians(0.038)} ${radians(0.211)}" />
         </joint>
         <joint name="${prefix_slave}gantry-${prefix_slave}kr16_joint" type="fixed">
@@ -46,4 +47,5 @@
             <parent link="${prefix_slave}tool0" />
             <child link="${prefix_slave}ktig_eef" />
+            <!-- <origin xyz="0.083 0.04227 0.44111" rpy="${radians(1.82)} ${radians(-42.9)} ${radians(-156.2)}" /> -->
             <origin xyz="0.0811 0.04116 0.4408" rpy="${radians(-179.61)} ${radians(-41.39)} ${radians(-153.95)}" />
             <!-- <origin xyz="0.121 0.05578 0.5307" rpy="${radians(0)} ${radians(-19.95)} ${radians(24.259)}" /> -->
@@ -65,8 +67,8 @@
             <origin xyz="1.1932095 0.8714369 0.3000" rpy="0.0 0.0 ${radians(0)}" />
         </joint> -->
-        <joint name="world_2-${prefix_master}positioner_side_joint" type="fixed">
+        <joint name="world-${prefix_master}positioner_side_joint" type="fixed">
             <parent link="world" />
             <child link="${prefix_master}positioner_side" />
-            <origin xyz="1.615 1.299017 -3.801712" rpy="0.0 0.0 0.0" />
+            <origin xyz="4.64146 2.53522 -8.77269" rpy="0.0 ${radians(0.13)} ${radians(-2.34)}" />
         </joint>
         <joint name="${prefix_master}positioner_side_joint-${prefix_master}positioner_joint" type="fixed">

Commit message: CMakeLists.txt for Kuka KR16

File: mimic_support/urdf/mimic_v2.xacro (robot description, xacro)
@@ -37,5 +37,5 @@
             <child link="${prefix_slave}gantry_frame" />
             <!-- <origin xyz="3.04787 1.209 -4.974558" rpy="0.0 ${radians(0.038)} ${radians(0.211)}" /> -->
-            <origin xyz="${3.05881-0.011} ${1.224-0.015} ${-4.98539-0.011}" rpy="0.0 ${radians(0.038)} ${radians(0.211)}" />
+            <origin xyz="${3.05881-0.011} ${1.224166-0.015} ${-4.98539307-0.011}" rpy="0.0 ${radians(0.038)} ${radians(0.211)}" />
         </joint>
         <joint name="${prefix_slave}gantry-${prefix_slave}kr16_joint" type="fixed">
