Commit message: Fix full driver RSI simulator and positioning based on robot's bases

File: mimic_support/urdf/mimic.xacro (robot description, xacro)
@@ -51,5 +51,6 @@
             <parent link="world" />
             <child link="world_2" />
-            <origin xyz="0.9183 0.721 -4.3402" rpy="0.0 0.0 0.0" />
+            <!-- <origin xyz="0.9183 0.721 -4.3402" rpy="0.0 0.0 0.0" /> -->
+            <origin xyz="1.568554 0.413247 -4.406904" rpy="0.0 0.0 0.0" />
         </joint>
         <joint name="world_2-${prefix_master}kr20_joint" type="fixed">
@@ -58,9 +59,15 @@
             <origin xyz="0 0 0" rpy="0.0 0.0 ${radians(-50)}" />
         </joint>
-        <joint name="world_2-${prefix_master}positioner_joint" type="fixed">
+        <!-- <joint name="world_2-${prefix_master}positioner_joint" type="fixed">
             <parent link="world_2" />
             <child link="${prefix_master}positioner_frame" />
+            <origin xyz="1.1932095 0.8714369 0.3000" rpy="0.0 0.0 ${radians(0)}" />
+        </joint> -->
+        <joint name="world-${prefix_master}positioner_joint" type="fixed">
+            <parent link="world" />
+            <child link="${prefix_master}positioner_frame" />
             <!-- <origin xyz="0.0994209235 1.4742 0.3000" rpy="0.0 0.0 ${radians(0)}" /> -->
-            <origin xyz="1.1932095 0.8714369 0.3000" rpy="0.0 0.0 ${radians(0)}" />
+            <!-- <origin xyz="1.1932095 0.8714369 0.3000" rpy="0.0 0.0 ${radians(0)}" /> -->
+            <origin xyz="2.1034488 1.68886 -3.996878" rpy="0.0 0.0 ${radians(0)}" />
         </joint>
     </robot>

Commit message: Fix URDF positions

File: mimic_support/urdf/mimic.xacro (robot description, xacro)
@@ -46,5 +46,5 @@
             <parent link="${prefix_slave}tool0" />
             <child link="${prefix_slave}ktig_eef" />
-            <origin xyz="0.0811 0.04116 0.4408" rpy="${radians(-179.61)} ${radians(-41.39)} ${radians(-153.95)}" />
+            <origin xyz="0.083 0.04227 0.4411" rpy="${radians(1.82)} ${radians(-42.9)} ${radians(-156.2)}" />
             <!-- <origin xyz="0.121 0.05578 0.5307" rpy="${radians(0)} ${radians(-19.95)} ${radians(24.259)}" /> -->
         </joint>

File: mimic_support/urdf/mimic_v2.xacro (robot description, xacro)
@@ -37,5 +37,5 @@
             <child link="${prefix_slave}gantry_frame" />
             <!-- <origin xyz="3.04787 1.209 -4.974558" rpy="0.0 ${radians(0.038)} ${radians(0.211)}" /> -->
-            <origin xyz="3.05881 1.224 -4.98539" rpy="0.0 ${radians(0.038)} ${radians(0.211)}" />
+            <origin xyz="${3.05881-0.011} ${1.224-0.015} ${-4.98539-0.011}" rpy="0.0 ${radians(0.038)} ${radians(0.211)}" />
         </joint>
         <joint name="${prefix_slave}gantry-${prefix_slave}kr16_joint" type="fixed">

Commit message: Mimic urdf based on IONA data

File: mimic_support/urdf/mimic.xacro (robot description, xacro)
@@ -11,4 +11,6 @@
         <xacro:include filename="$(find kuka_kr16_support)/urdf/kr16_2_macro.xacro" />
         <xacro:kuka_kr16_2 prefix="${prefix_slave}"/>
+        <link name="world" />
+        <link name="${prefix_master}positioner_side" />
         <link name="${prefix_slave}ktig_eef">
             <inertial>
@@ -30,50 +32,34 @@
             </collision>
         </link>
-        <link name="world" />
-        <link name="world_2" />
-        <link name="${prefix_master}positioner_side" />
-        <joint name="world-${prefix_slave}gantry_joint" type="fixed">
+        <joint name="world-${prefix_master}positioner_side_joint" type="fixed">
             <parent link="world" />
+            <child link="${prefix_master}positioner_side" />
+            <origin xyz="0 0 0" rpy="0 0 0" />
+        </joint>
+        <joint name="${prefix_master}positioner_side-${prefix_master}base_link" type="fixed">
+            <parent link="${prefix_master}positioner_side" />
+            <child link="${prefix_master}base_link" />
+            <origin xyz="-0.7260644 -0.509355 -0.603812" rpy="9.5e-05 -0.00184 -0.90717" />
+        </joint>
+        <joint name="${prefix_master}positioner_side-${prefix_slave}gantry_frame" type="fixed">
+            <parent link="${prefix_master}positioner_side" />
             <child link="${prefix_slave}gantry_frame" />
-            <origin xyz="0.0 0.0 0.0" rpy="0.0 0.0 0.0" />
+            <origin xyz="-1.1385215 -1.267 3.768157" rpy="0.00804 -0.00685 -0.00807" />
         </joint>
-        <joint name="${prefix_slave}gantry-${prefix_slave}kr16_joint" type="fixed">
-            <parent link="${prefix_slave}gantry_z" />
+        <joint name="${prefix_master}positioner_side-${prefix_master}positioner_frame" type="fixed">
+            <parent link="${prefix_master}positioner_side" />
+            <child link="${prefix_master}positioner_frame" />
+            <origin xyz="0.48839 0.390 -0.195" rpy="0.0 0.0 ${radians(0)}" />
+        </joint>
+        <joint name="${prefix_slave}gantry_frame-${prefix_slave}base_link" type="fixed">
+            <parent link="${prefix_slave}gantry_frame" />
             <child link="${prefix_slave}base_link" />
-            <origin xyz="0.0 0.0 0.0" rpy="${pi} 0.0 0.0" />
+            <origin xyz="0 0 0" rpy="${pi} 0 0" />
         </joint>
-        <joint name="${prefix_slave}kr16-${prefix_slave}ktig_joint" type="fixed">
+        <joint name="${prefix_slave}tool0-${prefix_slave}ktig_eef" type="fixed">
             <parent link="${prefix_slave}tool0" />
             <child link="${prefix_slave}ktig_eef" />
-            <origin xyz="0.083 0.04227 0.4411" rpy="${radians(1.82)} ${radians(-42.9)} ${radians(-156.2)}" />
-            <!-- <origin xyz="0.121 0.05578 0.5307" rpy="${radians(0)} ${radians(-19.95)} ${radians(24.259)}" /> -->
-        </joint>
-        <joint name="world-world_2" type="fixed">
-            <parent link="world" />
-            <child link="world_2" />
-            <!-- <origin xyz="0.9183 0.721 -4.3402" rpy="0.0 0.0 0.0" /> -->
-            <origin xyz="1.568554 0.413247 -4.406904" rpy="0.0 0.0 0.0" />
-        </joint>
-        <joint name="world_2-${prefix_master}kr20_joint" type="fixed">
-            <parent link="world_2" />
-            <child link="${prefix_master}base_link" />
-            <origin xyz="0 0 0" rpy="0.0 0.0 ${radians(-50)}" />
-        </joint>
-        <!-- <joint name="world_2-${prefix_master}positioner_joint" type="fixed">
-            <parent link="world_2" />
-            <child link="${prefix_master}positioner_frame" />
-            <origin xyz="1.1932095 0.8714369 0.3000" rpy="0.0 0.0 ${radians(0)}" />
-        </joint> -->
-        <joint name="world_2-${prefix_master}positioner_side_joint" type="fixed">
-            <parent link="world" />
-            <child link="${prefix_master}positioner_side" />
-            <origin xyz="1.615 1.299017 -3.801712" rpy="0.0 0.0 0.0" />
-        </joint>
-        <joint name="${prefix_master}positioner_side_joint-${prefix_master}positioner_joint" type="fixed">
-            <parent link="${prefix_master}positioner_side" />
-            <child link="${prefix_master}positioner_frame" />
-            <!-- <origin xyz="0.0994209235 1.4742 0.3000" rpy="0.0 0.0 ${radians(0)}" /> -->
-            <!-- <origin xyz="1.1932095 0.8714369 0.3000" rpy="0.0 0.0 ${radians(0)}" /> -->
-            <origin xyz="0.48839 0.390 -0.195" rpy="0.0 0.0 ${radians(0)}" />
+            <!-- we should get these values from tool on Kuka pendant -->
+            <origin xyz="0.0811 0.04116 0.4408" rpy="${radians(-179.61)} ${radians(-41.39)} ${radians(-153.95)}" />
         </joint>
     </robot>

Commit message: Fixed gantry positions

File: mimic_support/urdf/mimic.xacro (robot description, xacro)
@@ -45,5 +45,6 @@
             <parent link="${prefix_master}positioner_side" />
             <child link="${prefix_slave}gantry_frame" />
-            <origin xyz="-1.1385215 -1.267 3.768157" rpy="0.00804 -0.00685 -0.00807" />
+            <!-- <origin xyz="-1.1385215 -1.267 3.768157" rpy="0.00804 -0.00685 -0.00807" /> -->
+            <origin xyz="-1.6454453024932296 -1.252142034197534 3.779355489407589" rpy="0.00804 -0.00685 -0.0080815" />
         </joint>
         <joint name="${prefix_master}positioner_side-${prefix_master}positioner_frame" type="fixed">
@@ -53,5 +54,5 @@
         </joint>
         <joint name="${prefix_slave}gantry_frame-${prefix_slave}base_link" type="fixed">
-            <parent link="${prefix_slave}gantry_frame" />
+            <parent link="${prefix_slave}gantry_z" />
             <child link="${prefix_slave}base_link" />
             <origin xyz="0 0 0" rpy="${pi} 0 0" />
@@ -61,5 +62,37 @@
             <child link="${prefix_slave}ktig_eef" />
             <!-- we should get these values from tool on Kuka pendant -->
-            <origin xyz="0.0811 0.04116 0.4408" rpy="${radians(-179.61)} ${radians(-41.39)} ${radians(-153.95)}" />
+            <!-- <origin xyz="0.0811 0.04116 0.4408" rpy="${radians(-179.61)} ${radians(-41.39)} ${radians(-153.95)}" /> -->
+            <origin xyz="0.09142 0.04817 0.43987" rpy="${radians(-180.79)} ${radians(-48.46)} ${radians(-153.76)}" />
         </joint>
+        <link name="test_positioner_side" />
+        <link name="test_slave_tool0" />
+        <link name="test_slave_base_link" />
+        <link name="test_slave_gantry_frame" />
+        <joint name="world-test_positioner_side" type="fixed">
+            <parent link="world" />
+            <child link="test_positioner_side" />
+            <origin xyz="0 0 0" rpy="0 0 0"  />
+        </joint>
+        <joint name="test_positioner_side-test_tool0" type="fixed">
+            <parent link="test_positioner_side" />
+            <child link="test_slave_tool0" />
+            <origin xyz="-0.258976 0.4061174 0.6052054" rpy="${radians(-154.819)} ${radians(38.9068)} ${radians(-146.213)}"  />
+        </joint>
+        <joint name="test_slave_tool0-test_slave_base_link" type="fixed">
+            <parent link="test_slave_tool0" />
+            <child link="test_slave_base_link" />
+            <origin xyz="-1.03932 0.11033 -1.253455" rpy="0.052877306944842856 -0.7816220773823008 -2.7196170270177986"  />
+        </joint>
+        <joint name="test_slave_base_link-test_slave_gantry_frame" type="fixed">
+            <parent link="test_slave_base_link" />
+            <child link="test_slave_gantry_frame" />
+            <origin xyz="-1.10918 2.24999 -1.70100" rpy="0.0 0.0 0.0"  />
+        </joint>
+<!--
+        positioner side to slave base link
+        -0.5065105324997785, 1.0023177751521826, 2.1041316744423137
+        positioner side to gantry_frame
+        -0.50651 - 1.10918 + 0.011 = -1.60469
+        1.002317 - 2.24999 + 0.015 = -1.232673
+        2.104132 + 1.70100 + 0.011 = 3.816132 -->
     </robot>

Commit message: Visual fixed

File: mimic_support/urdf/mimic.xacro (robot description, xacro)
@@ -65,6 +65,6 @@
             <origin xyz="0.09142 0.04817 0.43987" rpy="${radians(-180.79)} ${radians(-48.46)} ${radians(-153.76)}" />
         </joint>
-        <link name="test_positioner_side" />
-        <link name="test_slave_tool0" />
+        <!-- <link name="test_positioner_side" /> -->
+        <!-- <link name="test_slave_tool0" />
         <link name="test_slave_base_link" />
         <link name="test_slave_gantry_frame" />
@@ -88,5 +88,5 @@
             <child link="test_slave_gantry_frame" />
             <origin xyz="-1.10918 2.24999 -1.70100" rpy="0.0 0.0 0.0"  />
-        </joint>
+        </joint> -->
 <!--
         positioner side to slave base link
