Commit message: Makes basic kr16 moveit config

File: kuka_kr16_moveit_config/config/gazebo_kuka_kr16_2.urdf (robot description, URDF)
Before this commit: robot kuka_kr16_2, 10 links, 9 joints
Links:
- removed link flange
- link base_link: mass 2500 -> 2
Joints:
- removed joint flange-tool0
- removed joint joint_a6-flange
- added joint joint_a6-tool0: type fixed, parent link_6, child tool0, origin xyz=0.158 0 0 rpy=0 1.5707963267948966 0
- joint joint_a1: limit lower=-3.2288591161895095 upper=3.2288591161895095 effort=2500 velocity=2.722713633111154 -> lower=-3.2288591161895095 upper=3.2288591161895095 effort=0 velocity=2.722713633111154
- joint joint_a2: limit lower=-2.705260340591211 upper=0.6108652381980153 effort=3100 velocity=2.722713633111154 -> lower=-2.705260340591211 upper=0.6108652381980153 effort=0 velocity=2.722713633111154
- joint joint_a3: limit lower=-2.2689280275926285 upper=2.6878070480712677 effort=2200 velocity=2.722713633111154 -> lower=-2.2689280275926285 upper=2.6878070480712677 effort=0 velocity=2.722713633111154
- joint joint_a4: limit lower=-6.1086523819801535 upper=6.1086523819801535 effort=500 velocity=5.759586531581287 -> lower=-6.1086523819801535 upper=6.1086523819801535 effort=0 velocity=5.759586531581287
- joint joint_a5: limit lower=-2.2689280275926285 upper=2.2689280275926285 effort=500 velocity=5.759586531581287 -> lower=-2.2689280275926285 upper=2.2689280275926285 effort=0 velocity=5.759586531581287
- joint joint_a6: limit lower=-6.1086523819801535 upper=6.1086523819801535 effort=150 velocity=10.733774899765127 -> lower=-6.1086523819801535 upper=6.1086523819801535 effort=0 velocity=10.733774899765127
